File: pcb/dialpad.kicad_pcb (KiCad board)
At the start: 2 copper layers, 100 x 92 mm, 21 parts, among them J1 Conn_01x04_Pin, SW1 SW_Push, SW10 RotaryEncoder_Switch, SW2 SW_Push, SW3 SW_Push, SW4 SW_Push, SW5 SW_Push, SW6 SW_Push, SW7 SW_Push, SW8 SW_Push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

Commit message: add firmware and touch ups on PCB
Parts:
- U1: value XIAO-RP2350-DIP -> XIAO-RP2040-DIP
Changed lines of the file:
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@@
 			)
 		)
-		(property "Value" "XIAO-RP2350-DIP"
+		(property "Value" "XIAO-RP2040-DIP"
 			(at 0 0 0)
 			(unlocked yes)
@@
 		)
 		(fp_line
-			(start -4.495 -10.541)
-			(end -4.491272 -11.451272)
-			(stroke
-				(width 0.127)
-				(type solid)
-			)
-			(layer "F.SilkS")
-		)
-		(fp_line
-			(start -3.991272 -11.951)
-			(end 4.004 -11.951)
-			(stroke
-				(width 0.127)
-				(type solid)
-			)
-			(layer "F.SilkS")
-		)
-		(fp_line
-			(start 4.504 -11.451)
-			(end 4.504 -10.541)
-			(stroke
-				(width 0.127)
-				(type solid)
-			)
-			(layer "F.SilkS")
-		)
-		(fp_line
 			(start 6.985 -10.541)
 			(end -6.985 -10.541)
@@
 			)
 			(layer "F.SilkS")
-		)
-		(fp_arc
-			(start -4.491272 -11.451272)
-			(mid -4.344728 -11.80464)
-			(end -3.991272 -11.951)
-			(stroke
-				(width 0.127)
-				(type default)
-			)
-			(layer "F.SilkS")
-		)
-		(fp_arc
-			(start 4.004 -11.951)
-			(mid 4.357553 -11.804553)
-			(end 4.504 -11.451)
-			(stroke
-				(width 0.127)
-				(type default)
-			)
-			(layer "F.SilkS")
