File: pcb/dialpad.kicad_sch (KiCad schematic)
At the start: 21 parts, among them J1 Conn_01x04_Pin, SW1 SW_Push, SW10 RotaryEncoder_Switch, SW2 SW_Push, SW3 SW_Push, SW4 SW_Push, SW5 SW_Push, SW6 SW_Push, SW7 SW_Push, SW8 SW_Push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

Commit message: add firmware and touch ups on PCB
Parts:
- U1: value XIAO-RP2350-DIP -> XIAO-RP2040-DIP
Changed lines of the file:
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@@
 			)
 		)
-		(property "Value" "XIAO-RP2350-DIP"
+		(property "Value" "XIAO-RP2040-DIP"
 			(at 148.59 50.8 0)
 			(effects
